File: PCB/TMC6300_BLDC.kicad_sch (KiCad schematic)
At the start: 14 parts, among them J2 Conn_01x03, U4 TMC6300-LA-T_C5274455

Commit message: Uploaded to JLC - ordering
Other:
- note added: "Next iteration needs a new BLDC driver; TMC6300 is out of stock on LCSC."
Changed lines of the file:
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@@
 	(generator_version "9.0")
 	(paper "A4")
+	(text "Next iteration needs a new BLDC driver;\nTMC6300 is out of stock on LCSC."
+		(exclude_from_sim no)
+		(at 133.096 72.898 0)
+		(effects
+			(font
+				(size 1.27 1.27)
+			)
+		)
+	)
 	(junction
 		(at 104.14 97.79)
