File: PCB/detentOne.kicad_pcb (KiCad board)
At the start: 4 copper layers, 150 x 85 mm, 97 parts, among them J1 Conn_01x07, J2 Conn_01x03, J5 Conn_01x05, J6 Conn_01x02, SW1 SW_Push, SW2 SW_Push, SW3 SW_Push, SW4 SW_Push, SW5 SW_Push, SW6 SW_Push, SW7 C92589, SW8 C92589, U1 ESP32-S3-WROOM-1U-N16R8, U2 SGM2050XTRL20G/TR, U4 TMC6300-LA-T_C5274455, U5 XY-GH1.25-7A61, U6 PCA9554ARGVR, U7 AS5047P-ATSM_C962063

Commit message: final checks for PCB, nearly ready to order v1
Parts:
- added R2: 22, Resistor_SMD:R_0402_1005Metric_Pad0.72x0.64mm_HandSolder, F.Cu at (154.9, 108.3)
- C9: value 10uF 10V -> 47uF; footprint Capacitor_SMD:C_0402_1005Metric -> Capacitor_SMD:C_0603_1608Metric
- R9: value 47K -> 10K
- moved C9 0.49 mm to (133.5, 95.2)
- moved C10 0.20 mm to (134.0, 93.9)
Connections:
- D5 pad 5: 3V3 -> 5V
- U1 pad 21: SCK -> Net-(U1-IO13)
- USB1 pad 13: unconnected-(USB1-SHELL-Pad13) -> GND
- USB1 pad 14: unconnected-(USB1-SHELL-Pad14) -> GND
Routing:
- net 3V3: track 118.3 -> 112.5 mm, vias 51 -> 50
- net 5V: track 94.9 -> 97.2 mm, vias 23 -> 24
- net Net-(U1-IO13): track 0.00 -> 2.11 mm
- net SCK: track 242.5 -> 240.7 mm
- net MOSI: track 218.8 -> 220.1 mm
- net ENCODER_CS: track 62.5 -> 63.4 mm
- net GND: track 55.3 -> 55.1 mm, vias 420 -> 424
Other:
- board text removed: "Add bulk capacitance to 5V in"

Commit message: Uploaded to JLC - ordering
Parts:
- C9: footprint Capacitor_SMD:C_0603_1608Metric -> Capacitor_SMD:C_0805_2012Metric
- moved C9 0.30 mm to (133.3, 95.4)
Routing:
- net W: track 34.0 -> 34.6 mm
- net GND: track 55.1 -> 55.2 mm, vias 424 -> 427
Changed lines of the file:
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@@
 		)
 	)
-	(footprint "Capacitor_SMD:C_0603_1608Metric"
+	(footprint "Capacitor_SMD:C_0805_2012Metric"
 		(layer "F.Cu")
-		(at 133.52 95.2 180)
-		(descr "Capacitor SMD 0603 (1608 Metric), square (rectangular) end terminal, IPC-7351 nominal, (Body size source: IPC-SM-782 page 76, https://www.pcb-3d.com/wordpress/wp-content/uploads/ipc-sm-782a_amendment_1_and_2.pdf), generated with kicad-footprint-generator")
+		(at 133.3 95.4 180)
+		(descr "Capacitor SMD 0805 (2012 Metric), square (rectangular) end terminal, IPC-7351 nominal, (Body size source: IPC-SM-782 page 76, https://www.pcb-3d.com/wordpress/wp-content/uploads/ipc-sm-782a_amendment_1_and_2.pdf, https://docs.google.com/spreadsheets/d/1BsfQQcO9C6DZCsRaXUlFlo91Tg2WpOkGARC1WS5S8t0/edit?usp=sharing), generated with kicad-footprint-generator")
 		(tags "capacitor")
 		(property "Reference" "C9"
-			(at 2.42 -0.1 180)
+			(at 0 -1.68 180)
 			(layer "F.SilkS")
 			(effects
@@
 		)
 		(property "Value" "47uF"
-			(at 0 1.43 180)
+			(at 0 1.68 180)
 			(layer "F.Fab")
-			(hide yes)
 			(effects
 				(font
@@
 		(attr smd)
 		(fp_line
-			(start -0.14058 0.51)
-			(end 0.14058 0.51)
+			(start -0.261252 0.735)
+			(end 0.261252 0.735)
 			(stroke
 				(width 0.12)
@@
 		)
 		(fp_line
-			(start -0.14058 -0.51)
-			(end 0.14058 -0.51)
+			(start -0.261252 -0.735)
+			(end 0.261252 -0.735)
 			(stroke
 				(width 0.12)
@@
 		)
 		(fp_rect
-			(start -1.48 -0.73)
-			(end 1.48 0.73)
+			(start -1.7 -0.98)
+			(end 1.7 0.98)
 			(stroke
 				(width 0.05)
@@
 		)
 		(fp_rect
-			(start -0.8 -0.4)
-			(end 0.8 0.4)
+			(start -1 -0.625)
+			(end 1 0.625)
 			(stroke
 				(width 0.1)
@@
 			(effects
 				(font
-					(size 0.4 0.4)
-					(thickness 0.06)
+					(size 0.5 0.5)
+					(thickness 0.08)
 				)
 			)
 		)
 		(pad "1" smd roundrect
-			(at -0.775 0 180)
-			(size 0.9 0.95)
+			(at -0.95 0 180)
+			(size 1 1.45)
 			(layers "F.Cu" "F.Mask" "F.Paste")
 			(roundrect_rratio 0.25)
@@
 		)
 		(pad "2" smd roundrect
-			(at 0.775 0 180)
-			(size 0.9 0.95)
+			(at 0.95 0 180)
+			(size 1 1.45)
 			(layers "F.Cu" "F.Mask" "F.Paste")
 			(roundrect_rratio 0.25)
@@
 		)
 		(embedded_fonts no)
-		(model "${KICAD9_3DMODEL_DIR}/Capacitor_SMD.3dshapes/C_0603_1608Metric.step"
+		(model "${KICAD9_3DMODEL_DIR}/Capacitor_SMD.3dshapes/C_0805_2012Metric.step"
 			(offset
 				(xyz 0 0 0)
@@
 	)
 	(segment
-		(start 135.79 94.71)
-		(end 135.79 95.04)
+		(start 135.79 95.01)
+		(end 135.275735 95.524265)
 		(width 0.2)
 		(layer "F.Cu")
@@
 	)
 	(segment
+		(start 135.79 94.71)
+		(end 135.999 94.71)
+		(width 0.2)
+		(layer "F.Cu")
+		(net 2)
+	)
+	(segment
 		(start 159 61.735)
 		(end 159.665 62.4)
@@
 	)
 	(segment
-		(start 135.79 95.04)
-		(end 135.23 95.6)
-		(width 0.2)
-		(layer "F.Cu")
-		(net 2)
-	)
-	(segment
 		(start 135.79 92.49)
 		(end 135.5 92.2)
@@
 	)
 	(segment
+		(start 135.79 94.71)
+		(end 135.79 95.01)
+		(width 0.2)
+		(layer "F.Cu")
+		(net 2)
+	)
+	(segment
 		(start 128.9 113.5)
 		(end 128.1 113.5)
@@
 	)
 	(via
+		(at 130.8 91.7)
+		(size 0.6)
+		(drill 0.3)
+		(layers "F.Cu" "B.Cu")
+		(net 2)
+	)
+	(via
 		(at 164.2 124.6)
 		(size 0.6)
@@
 	)
 	(via
-		(at 135.23 95.6)
-		(size 0.6)
-		(drill 0.3)
-		(layers "F.Cu" "B.Cu")
-		(net 2)
-	)
-	(via
 		(at 145.9 130)
 		(size 0.6)
@@
 	)
 	(via
+		(at 130.8 92.6)
+		(size 0.6)
+		(drill 0.3)
+		(layers "F.Cu" "B.Cu")
+		(net 2)
+	)
+	(via
 		(at 195.3 107)
 		(size 0.6)
@@
 	)
 	(via
+		(at 135.275735 95.524265)
+		(size 0.6)
+		(drill 0.3)
+		(layers "F.Cu" "B.Cu")
+		(net 2)
+	)
+	(via
 		(at 216.7 90.1)
 		(size 0.6)
@@
 	)
 	(via
+		(at 129.9 91.7)
+		(size 0.6)
+		(drill 0.3)
+		(layers "F.Cu" "B.Cu")
+		(net 2)
+	)
+	(via
 		(at 159.7 77.5)
 		(size 0.6)
@@
 	)
 	(segment
-		(start 132.401 96.601)
-		(end 135.119 96.601)
+		(start 131.3 96.5)
+		(end 131.401 96.601)
+		(width 0.2)
+		(layer "F.Cu")
+		(net 68)
+	)
+	(segment
+		(start 135.119 96.601)
+		(end 136.4 95.32)
 		(width 0.2)
 		(layer "F.Cu")
@@
 	)
 	(segment
-		(start 135.119 96.601)
-		(end 136.4 95.32)
+		(start 131.401 96.601)
+		(end 135.119 96.601)
 		(width 0.2)
 		(layer "F.Cu")
@@
 	(segment
 		(start 131.3 95.5)
-		(end 132.401 96.601)
+		(end 131.3 96.5)
 		(width 0.2)
 		(layer "F.Cu")
